File: Schematic_v1.brd (EAGLE design)
At the start: 30 x 30.5 mm, 15 parts, among them IC1 7805TV, J1 POWER_JACK, U1 ATTINY85-20P

Commit message: First version
Parts:
- moved J4 1.75 mm to (27.9, 25.4), turned to 269.8 degrees
Connections:
- net 5V: no longer J4.1
- net VOLT_IN: now also J4.1
Routing:
- net VOLT_IN: track 11.3 -> 23.4 mm
- net 5V: track 56.6 -> 50.3 mm
- net GND: track 23.6 -> 28.9 mm
- net PIN3: track 12.9 -> 11.1 mm
Other:
- board size 30 x 30.5 mm -> 30.5 x 30.5 mm
- board text added: "05102019"
- board text added: "VIN"
- board text removed: "PWR_1"
- board text removed: "PWR_2"
- board text removed: "RST_1"
- board text removed: "RST_2"
