File: Schematic_v1.sch (EAGLE design)
At the start: 15 parts, among them IC1 7805TV, J1 POWER_JACK, U1 ATTINY85-20P

Commit message: First version
Connections:
- net 5V: no longer J4.1
- net VOLT_IN: now also J4.1
Changed lines of the file:
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@@
 <?xml version="1.0" encoding="utf-8"?>
 <!DOCTYPE eagle SYSTEM "eagle.dtd">
-<eagle version="9.4.0">
+<eagle version="9.4.2">
 <drawing>
 <settings>
@@
 <label x="226.06" y="93.98" size="1.778" layer="95" rot="R90"/>
 </segment>
-<segment>
-<pinref part="J4" gate="G$1" pin="1"/>
-<wire x1="45.72" y1="88.9" x2="50.8" y2="88.9" width="0.1524" layer="91"/>
-<label x="48.26" y="88.9" size="1.778" layer="95"/>
-</segment>
 </net>
 <net name="VOLT_IN" class="0">
@@
 <label x="66.04" y="43.18" size="1.778" layer="95"/>
 </segment>
+<segment>
+<pinref part="J4" gate="G$1" pin="1"/>
+<wire x1="45.72" y1="88.9" x2="50.8" y2="88.9" width="0.1524" layer="91"/>
+<label x="48.26" y="88.9" size="1.778" layer="95"/>
+</segment>
 </net>
